Commit message: Update nexus_4wd_mecanum.xacro

File: nexus_4wd_mecanum_description/urdf/nexus_4wd_mecanum.xacro (robot description, xacro)
@@ -328,4 +328,31 @@
     </visual>
   </link>
+  <joint name="rplidar_joint" type="fixed">
+    <axis xyz="0 1 0" />
+    <origin xyz="0.165 0 0.058" rpy="0 0 3.14"/>
+    <parent link="base_link"/>
+    <child link="laser"/>
+  </joint>
+  <!-- rplidar Laser -->
+  <link name="laser">
+    <collision>
+      <origin xyz="0 0 0" rpy="1.5707 0 4.71"/>
+      <geometry>
+        <mesh filename="package://nexus_4wd_mecanum_description/meshes/rplidar.stl" scale="0.001 0.001 0.001" />
+      </geometry>
+    </collision>
+    <visual>
+      <origin xyz="0 0 0" rpy="1.5707 0 4.71"/>
+      <geometry>
+        <mesh filename="package://nexus_4wd_mecanum_description/meshes/rplidar.stl" scale="0.001 0.001 0.001" />
+      </geometry>
+      <material name="Black"/>
+    </visual>
+    <inertial>
+      <mass value="1e-5" />
+      <origin xyz="0 0 0" rpy="1.5707 0 4.71"/>
+      <inertia ixx="0" ixy="0" ixz="0" iyy="0" iyz="0" izz="0" />
+    </inertial>
+  </link>
   <!-- Include controller plugin for Gazebo -->
   <xacro:include filename="$(find nexus_4wd_mecanum_description)/urdf/nexus_4wd_mecanum.gazebo" />
